File: kicad/shield.sch (KiCad schematic (older format))
At the start: 44 parts, among them J1 Conn_01x12, J2 Conn_01x05, J3 Conn_01x03, J4 Conn_01x24, Q1 ZXMN3B01F, Q19 Q_PNP_BEC, Q29 Q_PNP_BEC, Q39 Q_PNP_BEC, SW1 SW_Push, SW2 SW_Push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

Commit message: replaced power LED with a PWM LED
Parts:
- removed D99: LED, LED_THT:LED_D3.0mm, symbol Device:LED
- removed R98: 1K, Resistor_SMD:R_0805_2012Metric_Pad1.15x1.40mm_HandSolder, symbol Device:R
- added D49: LED, LED_THT:LED_D3.0mm, symbol Device:LED
- added Q49: Q_PNP_BEC, Package_TO_SOT_SMD:SOT-23, symbol Device:Q_PNP_BEC
- added R48: 220, Resistor_SMD:R_0805_2012Metric_Pad1.15x1.40mm_HandSolder, symbol Device:R
- added R49: 1K, Resistor_SMD:R_0805_2012Metric_Pad1.15x1.40mm_HandSolder, symbol Device:R
Connections:
- net GND: now also D49.1 (K)
- net GPIO12_PWM0_BACKLIGHT: now also R49.1
- net P3V3: now also Q49.2 (E)
- new net: Q49.1 (B), R49.2
- new net: Q49.3 (C), R48.2
- new net: D49.2 (A), R48.1
Other:
- note added: "Pin 1, reserved 5 Volt"
- note removed: "Pin 1, reserved for 5 Volt"
- moved on the sheet: C39, D39, J3, Q39, R38, R39
Changed lines of the file:
@@
 L Device:Q_PNP_BEC Q39
 U 1 1 60C8825C
-P 12350 7750
-F 0 "Q39" H 12540 7704 50  0000 L CNN
-F 1 "Q_PNP_BEC" H 12540 7795 50  0000 L CNN
-F 2 "Package_TO_SOT_SMD:SOT-23" H 12550 7850 50  0001 C CNN
-F 3 "~" H 12350 7750 50  0001 C CNN
-	1    12350 7750
+P 12650 8350
+F 0 "Q39" H 12840 8304 50  0000 L CNN
+F 1 "Q_PNP_BEC" H 12840 8395 50  0000 L CNN
+F 2 "Package_TO_SOT_SMD:SOT-23" H 12850 8450 50  0001 C CNN
+F 3 "~" H 12650 8350 50  0001 C CNN
+	1    12650 8350
 	1    0    0    1
 $EndComp
@@
 L Device:R R39
 U 1 1 60CE4AF0
-P 11900 7750
-F 0 "R39" V 12000 7700 50  0000 L CNN
-F 1 "1K" V 11900 7700 50  0000 L CNN
-F 2 "Resistor_SMD:R_0805_2012Metric_Pad1.15x1.40mm_HandSolder" V 11830 7750 50  0001 C CNN
-F 3 "~" H 11900 7750 50  0001 C CNN
-	1    11900 7750
+P 12200 8350
+F 0 "R39" V 12300 8300 50  0000 L CNN
+F 1 "1K" V 12200 8300 50  0000 L CNN
+F 2 "Resistor_SMD:R_0805_2012Metric_Pad1.15x1.40mm_HandSolder" V 12130 8350 50  0001 C CNN
+F 3 "~" H 12200 8350 50  0001 C CNN
+	1    12200 8350
 	0    -1   -1   0
 $EndComp
 Wire Wire Line
-	12050 7750 12150 7750
+	12350 8350 12450 8350
 $Comp
 L Device:LED D39
 U 1 1 60D01AC1
-P 12450 8650
-F 0 "D39" V 12489 8533 50  0000 R CNN
-F 1 "LED" V 12398 8533 50  0000 R CNN
-F 2 "LED_THT:LED_D3.0mm" H 12450 8650 50  0001 C CNN
-F 3 "~" H 12450 8650 50  0001 C CNN
-	1    12450 8650
+P 12750 9250
+F 0 "D39" V 12789 9133 50  0000 R CNN
+F 1 "LED" V 12698 9133 50  0000 R CNN
+F 2 "LED_THT:LED_D3.0mm" H 12750 9250 50  0001 C CNN
+F 3 "~" H 12750 9250 50  0001 C CNN
+	1    12750 9250
 	0    1    -1   0
 $EndComp
 Wire Wire Line
-	12450 8500 12450 8350
-Wire Wire Line
-	12450 8900 12450 8800
+	12750 9100 12750 8950
+Wire Wire Line
+	12750 9500 12750 9400
 $Comp
 L Device:R R38
 U 1 1 610F3592
-P 12450 8200
-F 0 "R38" V 12550 8150 50  0000 L CNN
-F 1 "220" V 12450 8150 50  0000 L CNN
-F 2 "Resistor_SMD:R_0805_2012Metric_Pad1.15x1.40mm_HandSolder" V 12380 8200 50  0001 C CNN
-F 3 "~" H 12450 8200 50  0001 C CNN
-	1    12450 8200
+P 12750 8800
+F 0 "R38" V 12850 8750 50  0000 L CNN
+F 1 "220" V 12750 8750 50  0000 L CNN
+F 2 "Resistor_SMD:R_0805_2012Metric_Pad1.15x1.40mm_HandSolder" V 12680 8800 50  0001 C CNN
+F 3 "~" H 12750 8800 50  0001 C CNN
+	1    12750 8800
 	-1   0    0    1
 $EndComp
 Wire Wire Line
-	12450 8050 12450 7950
+	12750 8650 12750 8550
 $Comp
 L Connector_Generic:Conn_01x12 J1
@@
 $EndComp
 Wire Wire Line
-	9650 7850 10700 7850
-Wire Wire Line
-	10700 7850 10700 7300
-Wire Wire Line
-	10700 7300 12450 7300
-Wire Wire Line
-	12450 7300 12450 7550
-Wire Wire Line
-	12450 8900 10700 8900
-Wire Wire Line
-	10700 7950 10700 8900
-Wire Wire Line
-	9650 7950 10700 7950
-Text Label 9750 7850 0    50   ~ 0
+	9950 8450 11000 8450
+Wire Wire Line
+	11000 8450 11000 7900
+Wire Wire Line
+	11000 7900 12750 7900
+Wire Wire Line
+	12750 7900 12750 8150
+Wire Wire Line
+	12750 9500 11000 9500
+Wire Wire Line
+	11000 8550 11000 9500
+Wire Wire Line
+	9950 8550 11000 8550
+Text Label 10050 8450 0    50   ~ 0
 LED_Power
-Text Label 9750 7950 0    50   ~ 0
+Text Label 10050 8550 0    50   ~ 0
 LED_GND
 Wire Wire Line
-	9650 7750 11750 7750
+	9950 8350 12050 8350
 $Comp
 L Device:C C39
 U 1 1 5F43CD9B
-P 13400 8000
-F 0 "C39" H 13515 8046 50  0000 L CNN
-F 1 "0.1uF" H 13515 7955 50  0000 L CNN
-F 2 "Capacitor_SMD:C_0805_2012Metric" H 13438 7850 50  0001 C CNN
-F 3 "~" H 13400 8000 50  0001 C CNN
-	1    13400 8000
-	1    0    0    -1
-$EndComp
-Wire Wire Line
-	13400 7300 12450 7300
-Wire Wire Line
-	13400 7300 13400 7850
-Connection ~ 12450 7300
-Wire Wire Line
-	13400 8900 12450 8900
-Wire Wire Line
-	13400 8150 13400 8900
-Connection ~ 12450 8900
+P 13700 8600
+F 0 "C39" H 13815 8646 50  0000 L CNN
+F 1 "0.1uF" H 13815 8555 50  0000 L CNN
+F 2 "Capacitor_SMD:C_0805_2012Metric" H 13738 8450 50  0001 C CNN
+F 3 "~" H 13700 8600 50  0001 C CNN
+	1    13700 8600
+	1    0    0    -1
+$EndComp
+Wire Wire Line
+	13700 7900 12750 7900
+Wire Wire Line
+	13700 7900 13700 8450
+Connection ~ 12750 7900
+Wire Wire Line
+	13700 9500 12750 9500
+Wire Wire Line
+	13700 8750 13700 9500
+Connection ~ 12750 9500
 Wire Wire Line
 	850  10800 3400 10800
 Wire Wire Line
 	3400 10600 3400 10800
-Text Label 9750 7750 0    50   ~ 0
+Text Label 10050 8350 0    50   ~ 0
 GPIO16_Satus_LED_N
 $Comp
@@
 L Connector_Generic:Conn_01x03 J3
 U 1 1 6180A6AD
-P 9450 7850
-F 0 "J3" H 9368 7525 50  0000 C CNN
-F 1 "Conn_01x03" H 9368 7616 50  0000 C CNN
-F 2 "Connector_PinHeader_2.54mm:PinHeader_1x03_P2.54mm_Vertical" H 9450 7850 50  0001 C CNN
-F 3 "~" H 9450 7850 50  0001 C CNN
-	1    9450 7850
+P 9750 8450
+F 0 "J3" H 9668 8125 50  0000 C CNN
+F 1 "Conn_01x03" H 9668 8216 50  0000 C CNN
+F 2 "Connector_PinHeader_2.54mm:PinHeader_1x03_P2.54mm_Vertical" H 9750 8450 50  0001 C CNN
+F 3 "~" H 9750 8450 50  0001 C CNN
+	1    9750 8450
 	-1   0    0    1
 $EndComp
@@
 	1    0    0    -1
 $EndComp
-$Comp
-L Device:LED D99
-U 1 1 616DC77B
-P 12200 5300
-F 0 "D99" V 12239 5183 50  0000 R CNN
-F 1 "LED" V 12148 5183 50  0000 R CNN
-F 2 "LED_THT:LED_D3.0mm" H 12200 5300 50  0001 C CNN
-F 3 "~" H 12200 5300 50  0001 C CNN
-	1    12200 5300
+Text Label 12050 5000 0    50   ~ 0
+GPIO12_PWM0_BACKLIGHT
+Wire Wire Line
+	13050 5000 12050 5000
+$Comp
+L Device:Q_PNP_BEC Q49
+U 1 1 616B52AB
+P 13650 5000
+F 0 "Q49" H 13840 4954 50  0000 L CNN
+F 1 "Q_PNP_BEC" H 13840 5045 50  0000 L CNN
+F 2 "Package_TO_SOT_SMD:SOT-23" H 13850 5100 50  0001 C CNN
+F 3 "~" H 13650 5000 50  0001 C CNN
+	1    13650 5000
+	1    0    0    1
+$EndComp
+$Comp
+L Device:R R49
+U 1 1 616B52B5
+P 13200 5000
+F 0 "R49" V 13300 4950 50  0000 L CNN
+F 1 "1K" V 13200 4950 50  0000 L CNN
+F 2 "Resistor_SMD:R_0805_2012Metric_Pad1.15x1.40mm_HandSolder" V 13130 5000 50  0001 C CNN
+F 3 "~" H 13200 5000 50  0001 C CNN
+	1    13200 5000
+	0    -1   -1   0
+$EndComp
+Wire Wire Line
+	13350 5000 13450 5000
+$Comp
+L Device:LED D49
+U 1 1 616B52C0
+P 13750 5900
+F 0 "D49" V 13789 5783 50  0000 R CNN
+F 1 "LED" V 13698 5783 50  0000 R CNN
+F 2 "LED_THT:LED_D3.0mm" H 13750 5900 50  0001 C CNN
+F 3 "~" H 13750 5900 50  0001 C CNN
+	1    13750 5900
 	0    1    -1   0
 $EndComp
 Wire Wire Line
-	12200 5150 12200 5000
-Wire Wire Line
-	12200 5550 12200 5450
-$Comp
-L Device:R R98
-U 1 1 616DC787
-P 12200 4850
-F 0 "R98" V 12300 4800 50  0000 L CNN
-F 1 "1K" V 12200 4800 50  0000 L CNN
-F 2 "Resistor_SMD:R_0805_2012Metric_Pad1.15x1.40mm_HandSolder" V 12130 4850 50  0001 C CNN
-F 3 "~" H 12200 4850 50  0001 C CNN
-	1    12200 4850
+	13750 5750 13750 5600
+Wire Wire Line
+	13750 6150 13750 6050
+$Comp
+L Device:R R48
+U 1 1 616B52CC
+P 13750 5450
+F 0 "R48" V 13850 5400 50  0000 L CNN
+F 1 "220" V 13750 5400 50  0000 L CNN
+F 2 "Resistor_SMD:R_0805_2012Metric_Pad1.15x1.40mm_HandSolder" V 13680 5450 50  0001 C CNN
+F 3 "~" H 13750 5450 50  0001 C CNN
+	1    13750 5450
 	-1   0    0    1
 $EndComp
 Wire Wire Line
-	12200 4700 12200 4600
-$Comp
-L power:GND #PWR0103
-U 1 1 616DC792
-P 12200 5550
-F 0 "#PWR0103" H 12200 5300 50  0001 C CNN
-F 1 "GND" H 12200 5400 50  0000 C CNN
-F 2 "" H 12200 5550 50  0000 C CNN
-F 3 "" H 12200 5550 50  0000 C CNN
-	1    12200 5550
+	13750 5300 13750 5200
+Wire Wire Line
+	13750 4550 13750 4800
+$Comp
+L power:GND #PWR?
+U 1 1 616B52D8
+P 13750 6150
+F 0 "#PWR?" H 13750 5900 50  0001 C CNN
+F 1 "GND" H 13750 6000 50  0000 C CNN
+F 2 "" H 13750 6150 50  0000 C CNN
+F 3 "" H 13750 6150 50  0000 C CNN
+	1    13750 6150
 	-1   0    0    -1
 $EndComp
 Wire Wire Line
-	11200 4600 12200 4600
-Text Label 11200 4600 0    60   ~ 0
+	13300 4550 13750 4550
+Text Label 13300 4550 0    60   ~ 0
 P3V3
 Text Notes 3300 1350 0    50   ~ 0
-Pin 1, reserved for 5 Volt
+Pin 1, reserved 5 Volt
 $EndSCHEMATC
